File: Hardware/programming_board.kicad_pcb (KiCad board)
At the start: 2 copper layers, 45 x 70 mm, 41 parts, among them J1 Conn_02x03_Odd_Even, J10 Conn_02x03_Odd_Even, J11 Conn_01x05, J12 USB_C_Receptacle_USB2.0, J2 Conn_02x10_Odd_Even, J3 Conn_02x04_Odd_Even, J4 Conn_02x03_Odd_Even, J6 Conn_02x05_Odd_Even, J7 Conn_02x05_Odd_Even, J8 Conn_01x05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

Commit message: add stm8 programming connector; add 3d models
Parts:
- J1: value Conn_02x03_Odd_Even -> STM8_Prog_Conn; footprint custom:IDC-1.27-6P -> local:IDC-1.27-6P
- J10, J4: footprint custom:IDC-1.27-6P -> local:IDC-1.27-6P
- J2: footprint custom:IDC-Header_2x10_P2.54mm_Vertical -> local:IDC-Header_2x10_P2.54mm_Vertical
- J7: footprint custom:IDC-1.27-10P -> local:IDC-1.27-10P

Commit message: fix drc
Routing:
- net /BOOT: track 38.7 -> 55.9 mm, vias 4 -> 6
- net GND: track 418.6 -> 424.3 mm, vias 9 -> 10
- net /SWO: track 65.0 -> 66.5 mm

Commit message: Update programming_board.kicad_pcb
Parts:
- J10, J4: footprint local:IDC-1.27-6P -> custom:IDC-1.27-6P
- J2: footprint local:IDC-Header_2x10_P2.54mm_Vertical -> Connector_IDC:IDC-Header_2x10_P2.54mm_Vertical
- J7: footprint local:IDC-1.27-10P -> custom:IDC-1.27-10P
Other:
- board text added: "DAbramau"
